File: ps2-breakout.kicad_sch (KiCad schematic)
At the start: 33 parts, among them J1 Conn_01x08_Female, J2 Conn_01x08_Female, Q1 MMBF170, Q2 MMBF170, Q3 MMBF170, Q4 MMBF170, U1 RCLAMP0502A, U2 RCLAMP0502A, U3 MD-60SM, U4 MD-60SM

Commit message: Fix RCLAMP0502 symbol and footprint
Parts:
- DUAL CK1: renamed from DUAL-CK1
- DUAL DATA1: renamed from DUAL-DATA1
Connections:
- net +3V3: now also J2.1 (Pin_1)
- net GND: now also U1.2 (GND), U2.2 (GND); no longer J2.5 (Pin_5), U1.5 (GND), U2.5 (GND)
- net PS2_1.CLK: now also J2.3 (Pin_3); no longer J2.2 (Pin_2)
- net PS2_1.DATA: now also J2.2 (Pin_2); no longer J2.1 (Pin_1)
- net PS2_2.CLK: now also J2.5 (Pin_5); no longer J2.4 (Pin_4)
- net PS2_2.DATA: now also J2.4 (Pin_4); no longer J2.3 (Pin_3)
- net at FB1.2, TP9.1, U3.4 (VCC): now also U1.5 (VCC); no longer U1.2 (VCC)
- net at FB2.2, TP10.1, U4.4 (VCC): now also U2.5 (VCC); no longer U2.2 (VCC)
